Commit message: last changes on robot

File: strands_description/urdf/scitos_chest_camera.xacro (robot description, xacro)
@@ -28,5 +28,5 @@
     <!-- Z height from calibrate_chest -->
     <axis xyz="0 0 1"/>
-    <origin rpy="0 0 0" xyz="0.0294 0 0" />
+    <origin rpy="0 0 0" xyz="0.0594 0 0" />
     <limit effort="1000" velocity="1000" lower="0.5" upper="1.5"/>
     <parent link="base_link"/>
